Commit message: feat(cora_description): add collision sensor to cora model
- Added a collision sensor to `cora/base_link` in `cora.urdf.xacro`:
  - Defined a `<sensor>` of type `contact` to monitor collisions.
  - Configured the sensor to detect collisions on `cora/base_link_fixed_joint_lump__dummy_link_collision`.
  - Integrated the `gazebo_ros_bumper` plugin to publish collision states to the `cora/collision_sensor_states` topic.
  - Set the frame reference to `world` for proper alignment.

This update enhances the simulation by providing collision detection capabilities for the Cora model.

File: cora_description/urdf/cora.urdf.xacro (robot description, xacro)
@@ -45,3 +45,17 @@
     </inertial>
   </link>
+  <!-- Add collision sensor to base_link -->
+  <gazebo reference="cora/base_link">
+    <sensor type="contact" name="collision_sensor">
+      <always_on>true</always_on>
+      <update_rate>100.0</update_rate>
+      <contact>
+        <collision>cora/base_link_fixed_joint_lump__dummy_link_collision</collision>
+      </contact>
+      <plugin name="gazebo_ros_bumper" filename="libgazebo_ros_bumper.so">
+        <bumperTopicName>cora/collision_sensor_states</bumperTopicName>
+        <frameName>world</frameName>
+      </plugin>
+    </sensor>
+  </gazebo>
 </robot>

Commit message: feat(cora_description): improve collision sensor configuration for enhanced detection accuracy
- Updated the reference for the collision sensor from `cora/base_link` to `cora/dummy_link`.
- Increased the collision sensor `update_rate` from `100.0` to `500.0` for faster response.
- Corrected the collision target reference from `cora/base_link_fixed_joint_lump__dummy_link_collision` to `cora/dummy_link::collision`.
- Updated the `bumperTopicName` to `cora/sensors/collision` for better topic clarity and organization.
- Changed the `frameName` in the collision sensor plugin to `cora/dummy_link` for consistency.

These changes enhance the simulation's collision detection capability by improving sensor responsiveness and aligning configuration references with the model's structure.

File: cora_description/urdf/cora.urdf.xacro (robot description, xacro)
@@ -46,14 +46,14 @@
   </link>
   <!-- Add collision sensor to base_link -->
-  <gazebo reference="cora/base_link">
+  <gazebo reference="cora/dummy_link">
     <sensor type="contact" name="collision_sensor">
       <always_on>true</always_on>
-      <update_rate>100.0</update_rate>
+      <update_rate>500.0</update_rate>
       <contact>
-        <collision>cora/base_link_fixed_joint_lump__dummy_link_collision</collision>
+        <collision>cora/dummy_link::collision</collision>
       </contact>
       <plugin name="gazebo_ros_bumper" filename="libgazebo_ros_bumper.so">
-        <bumperTopicName>cora/collision_sensor_states</bumperTopicName>
-        <frameName>world</frameName>
+        <bumperTopicName>cora/sensors/collision</bumperTopicName>
+        <frameName>cora/dummy_link</frameName>
       </plugin>
     </sensor>
