Commit message: feat(cora_description): add dynamic thruster configuration for USV
- Updated `cora.xacro` to support dynamic thruster configuration selection (`H`, `M` layouts).
- Added `thrusters_h.xacro` and `thrusters_m.xacro` under `thrust_layouts/` to define specific thruster layouts.
- Integrated the `thruster_config` argument into `collision_avoidance.launch` for easier configuration.
- Adjusted `collision_avoidance.launch` to pass `thruster_config` to `cora.xacro` via the `robot_description` parameter.
- Enhanced flexibility and modularity for simulating various thruster layouts in the USV.

File: cora_description/urdf/cora.xacro (robot description, xacro)
@@ -1,19 +1,29 @@
 <?xml version="1.0"?>
 <robot xmlns:xacro="http://ros.org/wiki/xacro" name="cora">
+  <!-- Arguments -->
   <xacro:arg name="locked" default="false" />
-  <!-- Include macros for dynamics plugins -->
+  <xacro:arg name="thruster_config" default="" />
+  <xacro:arg name="namespace" default="cora" />
+  <xacro:arg name="thruster_namespace" default="thrusters/" />
+  <!-- Properties -->
+  <xacro:property name="namespace" value="$(arg namespace)" scope="global" />
+  <xacro:property name="thruster_namespace" value="$(arg thruster_namespace)" scope="global" />
+  <!-- Include Macros -->
   <xacro:include filename="$(find cora_description)/urdf/macros.xacro" />
-  <!-- Attach hydrodynamics plugin -->
+  <!-- Attach Hydrodynamics Plugin -->
   <xacro:usv_dynamics_gazebo name="cora_dynamics_plugin" />
-  <!-- Robot mesh -->
+  <!-- Robot Mesh -->
   <xacro:include filename="$(find cora_description)/urdf/cora.urdf.xacro" />
-  <!-- Note: this is only used for some sensors that do not correctly use the
-  robotNamespace parameter -->
-  <xacro:arg name="namespace" default="cora"/>
-  <xacro:property name="namespace" value="$(arg namespace)" scope="global" />
   <!-- Thrusters -->
-  <xacro:arg name="thruster_namespace" default="thrusters/"/>
-  <xacro:property name="thruster_namespace" value="$(arg thruster_namespace)" scope="global" />
-  <xacro:include filename="$(find cora_description)/urdf/thrusters.xacro" />
+  <!-- Add thrusters based on thruster_config variable -->
+  <xacro:property name="thruster_conf" value="$(arg thruster_config)" />
+  <!-- Default CORA with two aft thrusters (H configuration) -->
+  <xacro:if value="${thruster_conf == 'H'}">
+    <xacro:include filename="$(find cora_description)/urdf/thrust_layouts/thrusters_h.xacro" />
+  </xacro:if>
+  <xacro:if value="${thruster_conf == 'M'}">
+    <xacro:include filename="$(find cora_description)/urdf/thrust_layouts/thrusters_m.xacro" />
+  </xacro:if>
+  <!-- <xacro:include filename="$(find cora_description)/urdf/thrust_layouts/thrusters_h.xacro" /> -->
   <!-- Decide if we lock the robot to the world -->
   <xacro:if value="$(arg locked)">
